File: pcb/revA/revA.kicad_pcb (KiCad board)
At the start: 4 copper layers, 17.1 x 60.2 mm, 43 parts, among them J1 battery connector, J2 Conn_01x06, J3 USB_C_Receptacle, SW1 SW_Push, U1 charger, U2 buck, U3 MDBT50Q-1MV2, U4 AS7343, U5 MAX17048G+T10, U6 MX25R6435FZAIH0, U7 USBLC6-2SC6, Y1 32.768 kHz

Commit message: moved battery to the backside
Parts:
- added G***: LOGO, LOGO, F.Cu at (150.5, 53.2)
- J1: value battery connector -> SM02B-SRSS-TB; footprint Connector_JST:JST_PH_S2B-PH-SM4-TB_1x02-1MP_P2.00mm_Horizontal -> Connector_JST:JST_SH_SM02B-SRSS-TB_1x02-1MP_P1.00mm_Horizontal; moved to B.Cu
- moved J1 5.21 mm to (152.8, 49.6), turned to 180 degrees
Routing:
- net +BATT: track 26.2 -> 36.6 mm, vias 0 -> 1
Other:
- board text removed: "Sebastian Le & Emir Durakovic"
