File: pcb/revA/revA.kicad_pcb (KiCad board)
At the start: 4 copper layers, 17.1 x 60.2 mm, 44 parts, among them J1 SM02B-SRSS-TB, J2 Conn_01x06, J3 USB_C_Receptacle, SW1 SW_Push, U1 charger, U2 buck, U3 MDBT50Q-1MV2, U4 AS7343, U5 MAX17048G+T10, U6 MX25R6435FZAIH0, U7 USBLC6-2SC6, Y1 32.768 kHz

Commit message: outlined driver for AS7343
Parts:
- J1: footprint Connector_JST:JST_SH_SM02B-SRSS-TB_1x02-1MP_P1.00mm_Horizontal -> Connector_JST:JST_PH_S2B-PH-SM4-TB_1x02-1MP_P2.00mm_Horizontal
- moved J1 2.07 mm to (151.1, 50.8)
Routing:
- net +BATT: track 36.6 -> 31.5 mm
- net GND: track 59.1 -> 60.0 mm
- net /AS_INT: track 47.3 -> 47.9 mm
