File: pcb/revA/revA.kicad_sch (KiCad schematic)
At the start: 43 parts, among them J1 battery connector, J2 Conn_01x06, J3 USB_C_Receptacle, SW1 SW_Push, U1 charger, U2 buck, U3 MDBT50Q-1MV2, U4 AS7343, U5 MAX17048G+T10, U6 MX25R6435FZAIH0, U7 USBLC6-2SC6, Y1 32.768 kHz

Commit message: moved battery to the backside
Parts:
- J1: value battery connector -> SM02B-SRSS-TB; footprint Connector_JST:JST_PH_S2B-PH-SM4-TB_1x02-1MP_P2.00mm_Horizontal -> Connector_JST:JST_SH_SM02B-SRSS-TB_1x02-1MP_P1.00mm_Horizontal; LCSC C295747 -> (none); now left out of the parts list
Changed lines of the file:
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@@
 		(body_style 1)
 		(exclude_from_sim no)
-		(in_bom yes)
+		(in_bom no)
 		(on_board yes)
-		(in_pos_files yes)
+		(in_pos_files no)
 		(dnp no)
 		(fields_autoplaced yes)
@@
 			)
 		)
-		(property "Value" "battery connector"
+		(property "Value" "SM02B-SRSS-TB"
 			(at 71.12 34.2899 90)
 			(show_name no)
@@
 			)
 		)
-		(property "Footprint" "Connector_JST:JST_PH_S2B-PH-SM4-TB_1x02-1MP_P2.00mm_Horizontal"
+		(property "Footprint" "Connector_JST:JST_SH_SM02B-SRSS-TB_1x02-1MP_P1.00mm_Horizontal"
 			(at 68.58 33.02 0)
 			(hide yes)
@@
 			)
 		)
-		(property "LCSC" "C295747"
+		(property "LCSC" ""
 			(at 68.58 33.02 0)
 			(hide yes)

Commit message: outlined driver for AS7343
Parts:
- J1: footprint Connector_JST:JST_SH_SM02B-SRSS-TB_1x02-1MP_P1.00mm_Horizontal -> Connector_JST:JST_PH_S2B-PH-SM4-TB_1x02-1MP_P2.00mm_Horizontal; LCSC (none) -> C295747
Changed lines of the file:
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@@
 			)
 		)
-		(property "Footprint" "Connector_JST:JST_SH_SM02B-SRSS-TB_1x02-1MP_P1.00mm_Horizontal"
+		(property "Footprint" "Connector_JST:JST_PH_S2B-PH-SM4-TB_1x02-1MP_P2.00mm_Horizontal"
 			(at 68.58 33.02 0)
 			(hide yes)
@@
 			)
 		)
-		(property "LCSC" ""
+		(property "LCSC" "C295747"
 			(at 68.58 33.02 0)
 			(hide yes)
